Commit message: Detectron update

File: source/ext/objects/kettle/urdf/kettle.urdf (robot description, URDF)
Before this commit: robot cube.urdf, 1 links, 0 joints
Links:
- link baseLink: geometry collision mesh filename=./ext/objects/kettle/mesh/kettle.obj scale=.001 .001 .001; visual mesh filename=./ext/objects/kettle/mesh/kettle.obj scale=.001 .001 .001
