Commit message: add colision and mass to gripper and ee_link

File: source/ext/objects/ur10_robot/dependencies/ur_description/urdf/ur10_robot_with_graper.urdf (robot description, URDF)
Before this commit: robot ur10, 14 links, 13 joints
Links:
- link ee_link: mass None -> 0.05
- link gripper_link: mass None -> 0.4; geometry collision mesh filename=package://schunk_wsg50_model/meshes/wsg50_110.stl scale=0.001 0.001 0.001; visual mesh filename=package://schunk_wsg50_model/meshes/wsg50_110.stl scale=0.001 0.001 0.001
- link index_link: mass None -> 0.12; geometry collision mesh filename=package://schunk_wsg50_model/meshes/wsg_f.stl scale=0.001 0.001 0.001; visual mesh filename=package://schunk_wsg50_model/meshes/wsg_f.stl scale=0.001 0.001 0.001
- link thumb_link: mass None -> 0.12; geometry collision mesh filename=package://schunk_wsg50_model/meshes/wsg_f.stl scale=0.001 0.001 0.001; visual mesh filename=package://schunk_wsg50_model/meshes/wsg_f.stl scale=0.001 0.001 0.001

Commit message: delete mass for ee_link

File: source/ext/objects/ur10_robot/dependencies/ur_description/urdf/ur10_robot_with_graper.urdf (robot description, URDF)
Before this commit: robot ur10, 14 links, 13 joints
Links:
- link ee_link: mass 0.05 -> None

Commit message: MVP V.1.1
Созданы:

File: source/ext/objects/ur10_robot/dependencies/ur_description/urdf/ur10_robot_with_graper.urdf (robot description, URDF)
Before this commit: robot ur10, 14 links, 13 joints
Links:
- link ee_link: mass None -> 0.05
- link index_link: mass 0.12 -> 0.15
- link thumb_link: mass 0.12 -> 0.15
Joints:
- joint gripper_joint: origin xyz=0 0 0 rpy=-1.570796 0 0 -> xyz=0 0 0 rpy=-1.570796 0 -1.570796; parent ee_link -> tool0
- joint wrist_3_link-tool0_fixed_joint: origin xyz=0 0.0922 0 rpy=-1.57079632679 0 0 -> xyz=0 0.0922 0 rpy=-1.570796 0 0

Commit message: Исправлены баги

File: source/ext/objects/ur10_robot/dependencies/ur_description/urdf/ur10_robot_with_graper.urdf (robot description, URDF)
Before this commit: robot ur10, 14 links, 13 joints
Links:
- link gripper_link: mass 0.4 -> 0.9

Commit message: check grep

File: source/ext/objects/ur10_robot/dependencies/ur_description/urdf/ur10_robot_with_graper.urdf (robot description, URDF)
Before this commit: robot ur10, 14 links, 13 joints
Links:
- link ee_link: mass None -> 0.05
- link gripper_link: mass 0.4 -> 0.9
- link index_link: mass 0.12 -> 0.15
- link thumb_link: mass 0.12 -> 0.15
Joints:
- joint gripper_joint: origin xyz=0 0 0 rpy=-1.570796 0 0 -> xyz=0 0 0 rpy=-1.570796 0 -1.570796; parent ee_link -> tool0
- joint wrist_3_link-tool0_fixed_joint: origin xyz=0 0.0922 0 rpy=-1.57079632679 0 0 -> xyz=0 0.0922 0 rpy=-1.570796 0 0
