Commit message: set up new robot

File: source/ext/objects/robot/ur10-wsg50-realsense.urdf (robot description, URDF)
Before this commit: robot ur10, 19 links, 18 joints
Joints:
- joint wsg50_base_lip2_joint: limit lower=0 upper=0.055 effort=30 velocity=50 -> lower=0 upper=0.055 effort=30 velocity=0.5
